Commit message: add collision

File: urdf/accessories/rplidar_s2.urdf (robot description, URDF)
Before this commit: robot rplidar_s2, 1 links, 1 joints
Links:
- link lidar_link: geometry collision mesh filename=file://$(find myCode)/meshes/centered_rplidar-s1m1-r1.stl scale=0.001 0.001 0.001; visual mesh filename=file://$(find myCode)/meshes/centered_rplidar-s1m1-r1.stl scale=0.001 0.001 0.001
