Commit message: fix urdf

File: urdf/accessories/imu.urdf (robot description, URDF)
Before this commit: robot imu, 1 links, 1 joints
Links:
- link imu_link: geometry visual box size=0.015 0.010 0.008
Joints:
- joint imu_to_payload: origin xyz=0 0 0 rpy=0 0 0 -> xyz=0.0715 0 0.014 rpy=0 0 1.5708

File: urdf/accessories/rplidar_s2.urdf (robot description, URDF)
Before this commit: robot rplidar_s2, 1 links, 1 joints
Links:
- link lidar_link: geometry visual mesh filename=file://$(find myCode)/meshes/centered_rplidar-s1m1-r1.stl scale=0.001 0.001 0.001
Joints:
- joint lidar_to_payload: origin xyz=0.174 0 0.10 rpy=0 0 3.1415 -> xyz=0 0 0.093 rpy=0 0 0

File: urdf/mini.urdf (robot description, URDF)
Before this commit: robot rover_mini, 6 links, 5 joints
Links:
- link chassis_link: geometry collision mesh filename=file://$(find myCode)/meshes/mini_chassis.dae; visual mesh filename=file://$(find myCode)/meshes/mini_chassis.dae
- link fl_wheel_link: geometry collision mesh filename=file://$(find myCode)/meshes/hub_6.5in.dae; visual mesh filename=file://$(find myCode)/meshes/hub_6.5in.dae
- link fr_wheel_link: geometry collision mesh filename=file://$(find myCode)/meshes/hub_6.5in.dae; visual mesh filename=file://$(find myCode)/meshes/hub_6.5in.dae
- link rl_wheel_link: geometry collision mesh filename=file://$(find myCode)/meshes/hub_6.5in.dae; visual mesh filename=file://$(find myCode)/meshes/hub_6.5in.dae
- link rr_wheel_link: geometry collision mesh filename=file://$(find myCode)/meshes/hub_6.5in.dae; visual mesh filename=file://$(find myCode)/meshes/hub_6.5in.dae

Commit message: fix link

File: urdf/accessories/imu.urdf (robot description, URDF)
Before this commit: robot imu, 1 links, 1 joints
Links:
- link imu_link: geometry visual box size=0.010 0.015 0.008
Joints:
- joint imu_to_payload: origin xyz=0.0715 0 0.014 rpy=0 0 1.5708 -> xyz=0.0715 0 0.014 rpy=0 0 0

Commit message: add acc to imu

File: urdf/accessories/imu.urdf (robot description, URDF)
Before this commit: robot imu, 1 links, 1 joints
Joints:
- joint imu_to_payload: origin xyz=0.0715 0 0.014 rpy=0 0 0 -> xyz=0.0715 0 0.014 rpy=0 0 1.5457
