Commit message: before changes on urdf

File: urdf/mini.urdf (robot description, URDF)
Before this commit: robot rover_mini, 7 links, 6 joints
Links:
- removed link base_footprint
Joints:
- removed joint test_link

Commit message: fix for free fleet

File: urdf/mini.urdf (robot description, URDF)
Before this commit: robot rover_mini, 6 links, 5 joints
Links:
- added link base_footprint
Joints:
- added joint base_to_base_footprint: type fixed, parent base_link, child base_footprint, origin xyz=0 0 0
